File: schematics/tx_board/tx_board.sch (KiCad schematic (older format))
At the start: 16 parts, among them U1 SI4463-C2A-GM, X2 SMA

Commit message: first complete design & routing
Parts:
- removed C0: 8p2, tx_board:C0805, symbol tx_board-eagle-import:C-EUC0805
- removed C1: 1u/TA, tx_board:C1206, symbol tx_board-eagle-import:C-EUC1206
- removed C2: 10n, tx_board:C0805, symbol tx_board-eagle-import:C-EUC0805
- removed C3: 1n, tx_board:C0805, symbol tx_board-eagle-import:C-EUC0805
- removed CM1, CM2, CM3: 9p1, tx_board:C0805, symbol tx_board-eagle-import:C-EUC0805
- removed CM4: 13p, tx_board:C0805, symbol tx_board-eagle-import:C-EUC0805
- removed JP1: PINHD-2X5_90, tx_board:2X05_90, symbol tx_board-eagle-import:PINHD-2X5_90
- removed L0: 30nH, tx_board:R0805, symbol tx_board-eagle-import:R-EU_R0805
- removed LCHOKE1: 220nH, tx_board:R0805, symbol tx_board-eagle-import:R-EU_R0805
- removed LM1: 27nH, tx_board:R0805, symbol tx_board-eagle-import:R-EU_R0805
- removed LM2: 22nH, tx_board:R0805, symbol tx_board-eagle-import:R-EU_R0805
- removed LM3: 15nH, tx_board:R0805, symbol tx_board-eagle-import:R-EU_R0805
- removed U1: SI4463-C2A-GM, tx_board:QFN50P400X400X90-20N, symbol tx_board-eagle-import:SI4463-C2A-GM
- removed X2: SMA, tx_board:J502-ND-142-0701-871_876, symbol tx_board-eagle-import:SMA-142-0701-871_876
- added C301: 220p, Capacitor_SMD:C_0603_1608Metric_Pad1.05x0.95mm_HandSolder, symbol tx_board-rescue:C_Small-Device-Mainboard-rescue-rx_board-rescue-rx_board-rescue
- added C302: 10p, Capacitor_SMD:C_0603_1608Metric_Pad1.05x0.95mm_HandSolder, symbol tx_board-rescue:C_Small-Device-Mainboard-rescue-rx_board-rescue-rx_board-rescue
- added C303, C304, C307, C314, C318: 10n, Capacitor_SMD:C_0603_1608Metric_Pad1.05x0.95mm_HandSolder, symbol tx_board-rescue:C_Small-Device-Mainboard-rescue-rx_board-rescue-rx_board-rescue
- added C305: 2n2, Capacitor_SMD:C_0603_1608Metric_Pad1.05x0.95mm_HandSolder, symbol tx_board-rescue:C_Small-Device-Mainboard-rescue-rx_board-rescue-rx_board-rescue
- added C306, C308, C309, C315, C316: 100n, Capacitor_SMD:C_0603_1608Metric_Pad1.05x0.95mm_HandSolder, symbol tx_board-rescue:C_Small-Device-Mainboard-rescue-rx_board-rescue-rx_board-rescue
- added C310: 470p, Capacitor_SMD:C_0603_1608Metric_Pad1.05x0.95mm_HandSolder, symbol tx_board-rescue:C_Small-Device-Mainboard-rescue-rx_board-rescue-rx_board-rescue
- added C311: 22n, Capacitor_SMD:C_0603_1608Metric_Pad1.05x0.95mm_HandSolder, symbol tx_board-rescue:C_Small-Device-Mainboard-rescue-rx_board-rescue-rx_board-rescue
- added C312: 15n, Capacitor_SMD:C_0603_1608Metric_Pad1.05x0.95mm_HandSolder, symbol tx_board-rescue:C_Small-Device-Mainboard-rescue-rx_board-rescue-rx_board-rescue
- added C313: 1n, Capacitor_SMD:C_0603_1608Metric_Pad1.05x0.95mm_HandSolder, symbol tx_board-rescue:C_Small-Device-Mainboard-rescue-rx_board-rescue-rx_board-rescue
- added C317: 22u/TA, Capacitor_Tantalum_SMD:CP_EIA-3216-18_Kemet-A_Pad1.58x1.35mm_HandSolder, symbol tx_board-rescue:C_Small-device-Mainboard-rescue-rx_board-rescue-rx_board-rescue
- added C319: 6p8, Capacitor_SMD:C_0603_1608Metric_Pad1.05x0.95mm_HandSolder, symbol tx_board-rescue:C_Small-Device-Mainboard-rescue-rx_board-rescue-rx_board-rescue
- added C320: 1000p, Capacitor_SMD:C_0603_1608Metric_Pad1.05x0.95mm_HandSolder, symbol tx_board-rescue:C_Small-device-Mainboard-rescue-rx_board-rescue-rx_board-rescue
- added C321, C322: 9p1, Capacitor_SMD:C_0603_1608Metric_Pad1.05x0.95mm_HandSolder, symbol tx_board-rescue:C_Small-device-Mainboard-rescue-rx_board-rescue-rx_board-rescue
- added J1: Conn_02x14_Odd_Even, Connector_PinHeader_2.54mm:PinHeader_2x14_P2.54mm_Horizontal, symbol Connector_Generic:Conn_02x14_Odd_Even
- added J301: Out, Connector_Coaxial:SMA_Samtec_SMA-J-P-X-ST-EM1_EdgeMount, symbol tx_board-rescue:Conn_Coaxial-conn-Mainboard-rescue-rx_board-rescue-rx_board-res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
- added L301: 15n, Inductor_SMD:L_0603_1608Metric_Pad1.05x0.95mm_HandSolder, symbol tx_board-rescue:L_Small-Device-Mainboard-rescue-rx_board-rescue-rx_board-rescue
- added L302: DNP, Inductor_SMD:L_0603_1608Metric_Pad1.05x0.95mm_HandSolder, symbol tx_board-rescue:L_Small-Device-Mainboard-rescue-rx_board-rescue-rx_board-rescue
- added L303: 20n, Inductor_SMD:L_0603_1608Metric_Pad1.05x0.95mm_HandSolder, symbol tx_board-rescue:L_Small-Device-Mainboard-rescue-rx_board-rescue-rx_board-rescue
- added L304: 22n, Inductor_SMD:L_0603_1608Metric_Pad1.05x0.95mm_HandSolder, symbol tx_board-rescue:L_Small-Device-Mainboard-rescue-rx_board-rescue-rx_board-rescue
- added L305: 15nH, Inductor_SMD:L_0603_1608Metric_Pad1.05x0.95mm_HandSolder, symbol tx_board-rescue:L_Small-device-Mainboard-rescue-rx_board-rescue-rx_board-rescue
- added R301: 22k, Resistor_SMD:R_0603_1608Metric_Pad1.05x0.95mm_HandSolder, symbol tx_board-rescue:R_Small-Device-Mainboard-rescue-rx_board-rescue-rx_board-rescue
- added R302: 1k1, Resistor_SMD:R_0603_1608Metric_Pad1.05x0.95mm_HandSolder, symbol tx_board-rescue:R_Small-Device-Mainboard-rescue-rx_board-rescue-rx_board-rescue
- added R303, R306: 47k, Resistor_SMD:R_0603_1608Metric_Pad1.05x0.95mm_HandSolder, symbol tx_board-rescue:R_Small-Device-Mainboard-rescue-rx_board-rescue-rx_board-rescue
- added R304: 3k6, Resistor_SMD:R_0603_1608Metric_Pad1.05x0.95mm_HandSolder, symbol tx_board-rescue:R_Small-Device-Mainboard-rescue-rx_board-rescue-rx_board-rescue
- added R305: 3R9, Resistor_SMD:R_0603_1608Metric_Pad1.05x0.95mm_HandSolder, symbol tx_board-rescue:R_Small-Device-Mainboard-rescue-rx_board-rescue-rx_board-rescue
- added R307: 100, Resistor_SMD:R_0603_1608Metric_Pad1.05x0.95mm_HandSolder, symbol tx_board-rescue:R_Small-Device-Mainboard-rescue-rx_board-rescue-rx_board-rescue
- added R308: 560, Resistor_SMD:R_0603_1608Metric_Pad1.05x0.95mm_HandSolder, symbol tx_board-rescue:R_Small-Device-Mainboard-rescue-rx_board-rescue-rx_board-rescue
- added R309: 270, Resistor_SMD:R_0603_1608Metric_Pad1.05x0.95mm_HandSolder, symbol tx_board-rescue:R_Small-Device-Mainboard-rescue-rx_board-rescue-rx_board-rescue
- added RN301, RN302: 4 x 1k ISOLATED, Resistor_SMD:R_Array_Concave_4x0603, symbol Device:R_Pack04
- added TP301, TP302, TP303: TestPoint_Probe, TestPoint:TestPoint_Pad_D1.0mm, symbol tx_board-rescue:TestPoint_Probe-Connector-Mainboard-rescue-rx_board-rescue-rx_b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
- added U301: ADF7021, Package_CSP:LFCSP-48-1EP_7x7mm_P0.5mm_EP4.1x4.1mm_ThermalVias, symbol tx_board-rescue:ADF7021-adf7021-rx_board-rescue-rx_board-rescue
Connections:
- net +3V3: now also C301.1, C303.1, C304.1, C307.1, C314.1, C317.1, C318.1, J1.21 (Pin_21), J1.22 (Pin_22), L301.1, U301.3 (VDD1), U301.32 (VDD2), U301.40 (VDD3), U301.43 (VDD), U301.9 (VDD4)
- net GND: now also C301.2, C303.2, C304.2, C305.1, C306.2, C307.2, C309.2, C310.2, C312.2, C313.2, C314.2, C315.2, C316.1, C317.2, C318.2, C319.2, C321.1, C322.1, J1.1 (Pin_1), J1.11 (Pin_11), J1.12 (Pin_12), J1.19 (Pin_19), J1.2 (Pin_2), J1.20 (Pin_20), J1.23 (Pin_23), J1.24 (Pin_24), J1.27 (Pin_27), J1.28 (Pin_28), J1.5 (Pin_5), J1.6 (Pin_6), J301.2 (Ext), R301.1, R302.2, R304.2, U301.12 (GND4), U301.19 (GND4), U301.22 (GND4), U301.29 (GND2), U301.45 (GND), U301.47 (GND1), U301.49 (EPAD), U301.5 (RFGND)
- net TX: now also C302.1, L303.1
- new net: C322.2, J301.1 (In), L305.2
- new net: C320.1, C321.2, L305.1
- new net: C320.2, L304.2
- new net: R306.1, R307.2, TP301.1, U301.1 (VCOIN)
- new net: R304.1, U301.10 (RSET)
- new net: C309.1, U301.11 (CREG4)
- new net: C311.2, R305.1, U301.2 (CREG1)
- new net: RN301.4 (R4.1), U301.25 (SLE)
- new net: RN301.3 (R3.1), U301.26 (SDATA)
- new net: RN301.2 (R2.1), U301.27 (SREAD)
- new net: RN301.1 (R1.1), U301.28 (SCLK)
- new net: C316.2, U301.31 (CREG2)
- new net: RN302.4 (R4.1), U301.34 (TxRxDATA)
- new net: RN302.3 (R3.1), U301.35 (TxRxCLK)
- new net: RN302.2 (R2.1), U301.36 (CLKOUT)
- new net: RN302.1 (R1.1), U301.37 (MUXOUT)
- new net: C302.2, L301.2, U301.4 (RFOUT)
- new net: C315.1, U301.41 (CREG3)
- new net: C313.1, R308.1, R309.1, TP303.1, U301.42 (CPOUT)
- new net: L302.2, U301.44 (L2)
- new net: L302.1, U301.46 (L1)
- new net: C311.1, U301.48 (CVCO)
- new net: R302.1, U301.8 (RLNA)
- new net: C310.1, R307.1, R308.2, TP302.1
- new net: C308.1, R306.2
- new net: C305.2, C308.2, R303.2
- new net: C306.1, R305.2
- new net: C312.1, R309.2
- new net: C319.1, L303.2, L304.1
- new net ADF_CE: J1.17 (Pin_17), U301.24 (CE)
- new net ADF_MUXOUT: J1.8 (Pin_8), RN302.8 (R1.2)
- new net ADF_SCLK: J1.13 (Pin_13), RN301.8 (R1.2)
- new net ADF_SDATA: J1.15 (Pin_15), RN301.6 (R3.2)
- new net ADF_SLE: J1.18 (Pin_18), RN301.5 (R4.2)
- new net ADF_SREAD: J1.16 (Pin_16), RN301.7 (R2.2)
- new net ADF_SWD: J1.14 (Pin_14), U301.33 (SWD)
- new net EXT_OSC2_IN: J1.3 (Pin_3), J1.4 (Pin_4), U301.38 (OSC2)
- new net FM_MOD: J1.25 (Pin_25), J1.26 (Pin_26), R301.2, R303.1
- new net SPI2_MISO: J1.10 (Pin_10), RN302.6 (R3.2)
- new net SPI2_MOSI: J1.9 (Pin_9), RN302.5 (R4.2)
- new net SPI2_SCK: J1.7 (Pin_7), RN302.7 (R2.2)
- no-connect marks 0 -> 13
Other:
- note added: "Voltage at this point should be 0.2-2V"

Commit message: shielded version
Parts:
- added H1: Würt_LGA_Shielding, lib:WE_36103205_SMD, symbol Mechanical:MountingHole_Pad
- J1: footprint Connector_PinHeader_2.54mm:PinHeader_2x14_P2.54mm_Horizontal -> edge_contact:edge_2x14pin
Connections:
- net +3V3: now also J1.4 (Pin_4), J1.8 (Pin_8); no longer J1.21 (Pin_21), J1.22 (Pin_22)
- net ADF_CE: now also J1.1 (Pin_1); no longer J1.17 (Pin_17)
- net ADF_MUXOUT: now also J1.19 (Pin_19), J1.20 (Pin_20); no longer J1.8 (Pin_8)
- net ADF_SCLK: now also J1.9 (Pin_9); no longer J1.13 (Pin_13)
- net ADF_SDATA: now also J1.5 (Pin_5); no longer J1.15 (Pin_15)
- net ADF_SLE: now also J1.3 (Pin_3); no longer J1.18 (Pin_18)
- net ADF_SREAD: now also J1.7 (Pin_7); no longer J1.16 (Pin_16)
- net ADF_SWD: now also J1.11 (Pin_11), J1.12 (Pin_12); no longer J1.14 (Pin_14)
- net EXT_OSC2_IN: now also J1.23 (Pin_23), J1.24 (Pin_24); no longer J1.3 (Pin_3), J1.4 (Pin_4)
- net FM_MOD: now also J1.27 (Pin_27), J1.28 (Pin_28); no longer J1.25 (Pin_25), J1.26 (Pin_26)
- net GND: now also J1.10 (Pin_10), J1.21 (Pin_21), J1.22 (Pin_22), J1.25 (Pin_25), J1.26 (Pin_26), H1.1; no longer J1.1 (Pin_1), J1.11 (Pin_11), J1.12 (Pin_12), J1.19 (Pin_19), J1.20 (Pin_20), J1.23 (Pin_23), J1.24 (Pin_24), J1.27 (Pin_27), J1.28 (Pin_28), J1.5 (Pin_5)
- net SPI2_MISO: now also J1.15 (Pin_15), J1.16 (Pin_16); no longer J1.10 (Pin_10)
- net SPI2_MOSI: now also J1.13 (Pin_13), J1.14 (Pin_14); no longer J1.9 (Pin_9)
- net SPI2_SCK: now also J1.17 (Pin_17), J1.18 (Pin_18); no longer J1.7 (Pin_7)
Other:
- moved on the sheet: J1
Changed lines of the file:
@@
 	6200 3850 7600 3850
 NoConn ~ 6100 4850
+Text GLabel 7200 8550 3    50   Input ~ 0
+ADF_SLE
+Text GLabel 7300 8550 3    50   Input ~ 0
+ADF_SDATA
+Text GLabel 7400 8550 3    50   Input ~ 0
+ADF_SREAD
 Text GLabel 7500 8550 3    50   Input ~ 0
-ADF_SLE
-Text GLabel 7600 8050 1    50   Input ~ 0
-ADF_SDATA
+ADF_SCLK
 Text GLabel 7600 8550 3    50   Input ~ 0
-ADF_SREAD
-Text GLabel 7700 8050 1    50   Input ~ 0
-ADF_SCLK
+ADF_SWD
 Text GLabel 7700 8550 3    50   Input ~ 0
-ADF_SWD
-Text GLabel 7900 8050 1    50   Input ~ 0
 SPI2_MOSI
+Text GLabel 7800 8550 3    50   Input ~ 0
+SPI2_MISO
 Text GLabel 7900 8550 3    50   Input ~ 0
-SPI2_MISO
-Text GLabel 8000 8050 1    50   Input ~ 0
 SPI2_SCK
 Text GLabel 8000 8550 3    50   Input ~ 0
 ADF_MUXOUT
-Text GLabel 8200 8050 1    50   Input ~ 0
+Text GLabel 8200 8550 3    50   Input ~ 0
 EXT_OSC2_IN
-Text GLabel 7500 8050 1    50   Input ~ 0
+Text GLabel 7100 8550 3    50   Input ~ 0
 ADF_CE
-Text GLabel 7100 8550 3    50   Input ~ 0
+Text GLabel 8400 8550 3    50   Input ~ 0
 FM_MOD
 Wire Wire Line
-	7800 8050 7800 7950
-$Comp
-L power:GND #PWR09
-U 1 1 5F5CB5E7
-P 7800 7950
-F 0 "#PWR09" H 7800 7700 50  0001 C CNN
-F 1 "GND" H 7805 7777 50  0000 C CNN
-F 2 "" H 7800 7950 50  0001 C CNN
-F 3 "" H 7800 7950 50  0001 C CNN
-	1    7800 7950
-	-1   0    0    1
-$EndComp
-Wire Wire Line
-	7800 8550 7800 8650
-$Comp
-L power:GND #PWR010
-U 1 1 5F5D15A4
-P 7800 8650
-F 0 "#PWR010" H 7800 8400 50  0001 C CNN
-F 1 "GND" H 7805 8477 50  0000 C CNN
-F 2 "" H 7800 8650 50  0001 C CNN
-F 3 "" H 7800 8650 50  0001 C CNN
-	1    7800 8650
-	1    0    0    -1
-$EndComp
-Wire Wire Line
-	7400 8050 7400 7950
+	7500 8050 7500 7950
 $Comp
 L power:GND #PWR07
 U 1 1 5F5D7938
-P 7400 7950
-F 0 "#PWR07" H 7400 7700 50  0001 C CNN
-F 1 "GND" H 7405 7777 50  0000 C CNN
-F 2 "" H 7400 7950 50  0001 C CNN
-F 3 "" H 7400 7950 50  0001 C CNN
-	1    7400 7950
-	-1   0    0    1
-$EndComp
-Wire Wire Line
-	7200 8050 7200 7950
+P 7500 7950
+F 0 "#PWR07" H 7500 7700 50  0001 C CNN
+F 1 "GND" H 7505 7777 50  0000 C CNN
+F 2 "" H 7500 7950 50  0001 C CNN
+F 3 "" H 7500 7950 50  0001 C CNN
+	1    7500 7950
+	-1   0    0    1
+$EndComp
+Wire Wire Line
+	7300 8050 7300 7950
 $Comp
 L power:GND #PWR05
 U 1 1 5F5DDB86
-P 7200 7950
-F 0 "#PWR05" H 7200 7700 50  0001 C CNN
-F 1 "GND" H 7205 7777 50  0000 C CNN
-F 2 "" H 7200 7950 50  0001 C CNN
-F 3 "" H 7200 7950 50  0001 C CNN
-	1    7200 7950
-	-1   0    0    1
-$EndComp
-Wire Wire Line
-	7200 8550 7200 8650
-$Comp
-L power:GND #PWR06
-U 1 1 5F5E3E22
-P 7200 8650
-F 0 "#PWR06" H 7200 8400 50  0001 C CNN
-F 1 "GND" H 7205 8477 50  0000 C CNN
-F 2 "" H 7200 8650 50  0001 C CNN
-F 3 "" H 7200 8650 50  0001 C CNN
-	1    7200 8650
-	1    0    0    -1
-$EndComp
-Wire Wire Line
-	7400 8550 7400 8650
+P 7300 7950
+F 0 "#PWR05" H 7300 7700 50  0001 C CNN
+F 1 "GND" H 7305 7777 50  0000 C CNN
+F 2 "" H 7300 7950 50  0001 C CNN
+F 3 "" H 7300 7950 50  0001 C CNN
+	1    7300 7950
+	-1   0    0    1
+$EndComp
+Wire Wire Line
+	8300 8050 8300 7950
 $Comp
 L power:GND #PWR08
 U 1 1 5F5EA477
-P 7400 8650
-F 0 "#PWR08" H 7400 8400 50  0001 C CNN
-F 1 "GND" H 7405 8477 50  0000 C CNN
-F 2 "" H 7400 8650 50  0001 C CNN
-F 3 "" H 7400 8650 50  0001 C CNN
-	1    7400 8650
-	1    0    0    -1
-$EndComp
-Wire Wire Line
-	8100 8050 8100 7950
-$Comp
-L power:GND #PWR011
-U 1 1 5F5FE8B3
-P 8100 7950
-F 0 "#PWR011" H 8100 7700 50  0001 C CNN
-F 1 "GND" H 8105 7777 50  0000 C CNN
-F 2 "" H 8100 7950 50  0001 C CNN
-F 3 "" H 8100 7950 50  0001 C CNN
-	1    8100 7950
-	-1   0    0    1
-$EndComp
-Wire Wire Line
-	8300 8050 8300 7950
-$Comp
-L power:GND #PWR013
-U 1 1 5F604F03
 P 8300 7950
-F 0 "#PWR013" H 8300 7700 50  0001 C CNN
+F 0 "#PWR08" H 8300 7700 50  0001 C CNN
 F 1 "GND" H 8305 7777 50  0000 C CNN
 F 2 "" H 8300 7950 50  0001 C CNN
@@
 $EndComp
 Wire Wire Line
-	8200 8050 8250 8050
-Wire Wire Line
-	8250 8050 8250 8550
-Wire Wire Line
-	8250 8550 8200 8550
-Wire Wire Line
-	7000 8550 7000 8650
+	8100 8050 8100 7950
 $Comp
 L power:GND #PWR02
 U 1 1 5F63542E
-P 7000 8650
-F 0 "#PWR02" H 7000 8400 50  0001 C CNN
-F 1 "GND" H 7005 8477 50  0000 C CNN
-F 2 "" H 7000 8650 50  0001 C CNN
-F 3 "" H 7000 8650 50  0001 C CNN
-	1    7000 8650
-	1    0    0    -1
-$EndComp
-Wire Wire Line
-	7000 8050 7000 7950
+P 8100 7950
+F 0 "#PWR02" H 8100 7700 50  0001 C CNN
+F 1 "GND" H 8105 7777 50  0000 C CNN
+F 2 "" H 8100 7950 50  0001 C CNN
+F 3 "" H 8100 7950 50  0001 C CNN
+	1    8100 7950
+	-1   0    0    1
+$EndComp
+Wire Wire Line
+	7100 8050 7100 7950
 $Comp
 L power:GND #PWR01
 U 1 1 5F63C3C4
-P 7000 7950
-F 0 "#PWR01" H 7000 7700 50  0001 C CNN
-F 1 "GND" H 7005 7777 50  0000 C CNN
-F 2 "" H 7000 7950 50  0001 C CNN
-F 3 "" H 7000 7950 50  0001 C CNN
-	1    7000 7950
+P 7100 7950
+F 0 "#PWR01" H 7100 7700 50  0001 C CNN
+F 1 "GND" H 7105 7777 50  0000 C CNN
+F 2 "" H 7100 7950 50  0001 C CNN
+F 3 "" H 7100 7950 50  0001 C CNN
+	1    7100 7950
 	-1   0    0    1
 $EndComp
@@
 L power:+3.3V #PWR03
 U 1 1 5F64B16D
-P 7300 7950
-F 0 "#PWR03" H 7300 7800 50  0001 C CNN
-F 1 "+3.3V" H 7315 8123 50  0000 C CNN
-F 2 "" H 7300 7950 50  0001 C CNN
-F 3 "" H 7300 7950 50  0001 C CNN
-	1    7300 7950
-	1    0    0    -1
-$EndComp
-Wire Wire Line
-	7300 7950 7300 8050
+P 7400 7950
+F 0 "#PWR03" H 7400 7800 50  0001 C CNN
+F 1 "+3.3V" H 7415 8123 50  0000 C CNN
+F 2 "" H 7400 7950 50  0001 C CNN
+F 3 "" H 7400 7950 50  0001 C CNN
+	1    7400 7950
+	1    0    0    -1
+$EndComp
+Wire Wire Line
+	7400 7950 7400 8050
 $Comp
 L power:+3.3V #PWR04
 U 1 1 5F65259F
-P 7300 8650
-F 0 "#PWR04" H 7300 8500 50  0001 C CNN
-F 1 "+3.3V" H 7315 8823 50  0000 C CNN
-F 2 "" H 7300 8650 50  0001 C CNN
-F 3 "" H 7300 8650 50  0001 C CNN
-	1    7300 8650
-	-1   0    0    1
-$EndComp
-Wire Wire Line
-	7300 8650 7300 8550
+P 7200 7950
+F 0 "#PWR04" H 7200 7800 50  0001 C CNN
+F 1 "+3.3V" H 7215 8123 50  0000 C CNN
+F 2 "" H 7200 7950 50  0001 C CNN
+F 3 "" H 7200 7950 50  0001 C CNN
+	1    7200 7950
+	1    0    0    -1
+$EndComp
+Wire Wire Line
+	7200 7950 7200 8050
 $Comp
 L Connector_Generic:Conn_02x14_Odd_Even J1
 U 1 1 5F6643F7
-P 7700 8250
-F 0 "J1" V 7704 8930 50  0000 L CNN
-F 1 "Conn_02x14_Odd_Even" V 7795 8930 50  0000 L CNN
-F 2 "Connector_PinHeader_2.54mm:PinHeader_2x14_P2.54mm_Horizontal" H 7700 8250 50  0001 C CNN
-F 3 "~" H 7700 8250 50  0001 C CNN
-	1    7700 8250
-	0    1    1    0
-$EndComp
-Wire Wire Line
-	7100 8050 7100 8550
+P 7700 8350
+F 0 "J1" V 7704 9030 50  0000 L CNN
+F 1 "Conn_02x14_Odd_Even" V 7795 9030 50  0000 L CNN
+F 2 "edge_contact:edge_2x14pin" H 7700 8350 50  0001 C CNN
+F 3 "~" H 7700 8350 50  0001 C CNN
+	1    7700 8350
+	0    -1   -1   0
+$EndComp
+$Comp
+L Mechanical:MountingHole_Pad H1
+U 1 1 5F5F1835
+P 9850 2200
+F 0 "H1" H 9950 2249 50  0000 L CNN
+F 1 "Würt_LGA_Shielding" H 9950 2158 50  0000 L CNN
+F 2 "lib:WE_36103205_SMD" H 9850 2200 50  0001 C CNN
+F 3 "~" H 9850 2200 50  0001 C CNN
+	1    9850 2200
+	1    0    0    -1
+$EndComp
+$Comp
+L power:GND #PWR017
+U 1 1 5F5F2F75
+P 9850 2350
+F 0 "#PWR017" H 9850 2100 50  0001 C CNN
+F 1 "GND" H 9855 2177 50  0000 C CNN
+F 2 "" H 9850 2350 50  0001 C CNN
+F 3 "" H 9850 2350 50  0001 C CNN
+	1    9850 2350
+	1    0    0    -1
+$EndComp
+Wire Wire Line
+	9850 2300 9850 2350
+$Comp
+L power:GND #PWR016
+U 1 1 5F5FAC6F
+P 9500 2250
+F 0 "#PWR016" H 9500 2000 50  0001 C CNN
+F 1 "GND" H 9505 2077 50  0000 C CNN
+F 2 "" H 9500 2250 50  0001 C CNN
+F 3 "" H 9500 2250 50  0001 C CNN
+	1    9500 2250
+	1    0    0    -1
+$EndComp
+$Comp
+L power:PWR_FLAG #FLG02
+U 1 1 5F602B7C
+P 9500 2200
+F 0 "#FLG02" H 9500 2275 50  0001 C CNN
+F 1 "PWR_FLAG" H 9500 2373 50  0000 C CNN
+F 2 "" H 9500 2200 50  0001 C CNN
+F 3 "~" H 9500 2200 50  0001 C CNN
+	1    9500 2200
+	1    0    0    -1
+$EndComp
+$Comp
+L power:+3.3V #PWR015
+U 1 1 5F603595
+P 9050 2250
+F 0 "#PWR015" H 9050 2100 50  0001 C CNN
+F 1 "+3.3V" H 9065 2423 50  0000 C CNN
+F 2 "" H 9050 2250 50  0001 C CNN
+F 3 "" H 9050 2250 50  0001 C CNN
+	1    9050 2250
+	-1   0    0    1
+$EndComp
+$Comp
+L power:PWR_FLAG #FLG01
+U 1 1 5F60B0F9
+P 9050 2200
+F 0 "#FLG01" H 9050 2275 50  0001 C CNN
+F 1 "PWR_FLAG" H 9050 2373 50  0000 C CNN
+F 2 "" H 9050 2200 50  0001 C CNN
+F 3 "~" H 9050 2200 50  0001 C CNN
+	1    9050 2200
+	1    0    0    -1
+$EndComp
+Wire Wire Line
+	9050 2200 9050 2250
+Wire Wire Line
+	9500 2200 9500 2250
+Wire Wire Line
+	7600 8050 7600 8550
+Wire Wire Line
+	7700 8050 7700 8550
+Wire Wire Line
+	7900 8050 7900 8550
+Wire Wire Line
+	7800 8050 7800 8550
+Wire Wire Line
+	8000 8050 8000 8550
+Wire Wire Line
+	8200 8050 8200 8550
+Wire Wire Line
+	8400 8050 8400 8550
 $EndSCHEMATC
