File: schematics/pa_board/main_new.sch (KiCad schematic (older format))
At the start: 20 parts, among them J1 Conn_Coaxial, J2 Conn_Coaxial, X3 AK500_2, X4 AK500_2

Commit message: PA boad smd version, 50Ohms microstrip
Parts:
- removed C1, C2: 10u, main_new:E5-8,5, symbol main_new-eagle-import:CPOL-EUE5-8.5
- removed R1, R2: 8/0.8/5.0, main_new:0411_12, symbol main_new-eagle-import:R-EU_0411_12
- added C1, C2: 10uF, Capacitor_Tantalum_SMD:CP_EIA-7132-28_AVX-C_Pad2.72x3.50mm_HandSolder, symbol Device:CP_Small
- added L1, L2: 130nH, Lib:XEL3520131MEB, symbol Device:L_Small
- C3, C4, C5, C6: footprint main_new:C050-030X075 -> Capacitor_SMD:C_0805_2012Metric_Pad1.15x1.40mm_HandSolder
- X3, X4: footprint main_new:AK500_2 -> TerminalBlock_Phoenix:TerminalBlock_Phoenix_PT-1,5-2-5.0-H_1x02_P5.00mm_Horizontal
Connections:
- net GND: now also C1.2, C2.2
- net at C5.1, X4.2 (KL): now also L1.2
- net at C3.1, PAD2.1 (P): now also C1.1, L1.1
- net at C6.1, X3.2 (KL): now also L2.2
- net at C4.2, PAD3.1 (P): now also C2.1, L2.1
Changed lines of the file:
@@
 Wire Wire Line
 	7500 3700 7500 2800
-Wire Wire Line
-	7500 4100 7500 4000
-Wire Wire Line
-	7400 3700 7500 3700
 Connection ~ 7500 4000
 Connection ~ 7500 3700
 Wire Wire Line
-	6400 3700 6500 3700
-Wire Wire Line
-	6500 3700 6500 4000
-Wire Wire Line
-	6500 4000 6500 4100
-Wire Wire Line
 	6400 4000 6500 4000
-Wire Wire Line
-	6500 2800 6500 3700
-Connection ~ 6500 3700
 Connection ~ 6500 4000
 Wire Wire Line
 	6500 5300 6500 4600
-Wire Wire Line
-	6500 4600 6500 4500
 Wire Wire Line
 	6400 4600 6500 4600
@@
 Wire Wire Line
 	7500 4600 7400 4600
-Wire Wire Line
-	7500 4600 7500 4500
 Wire Wire Line
 	7500 5300 7500 4600
@@
 $EndComp
 $Comp
-L main_new-eagle-import:CPOL-EUE5-8.5 C1
-U 1 1 F3B28787
-P 6300 3700
-F 0 "C1" H 6345 3719 59  0000 L BNN
-F 1 "10u" H 6345 3519 59  0000 L BNN
-F 2 "main_new:E5-8,5" H 6300 3700 50  0001 C CNN
-F 3 "" H 6300 3700 50  0001 C CNN
-	1    6300 3700
-	0    1    1    0
-$EndComp
-$Comp
-L main_new-eagle-import:CPOL-EUE5-8.5 C2
-U 1 1 97363537
-P 7300 3700
-F 0 "C2" H 7345 3719 59  0000 L BNN
-F 1 "10u" H 7345 3519 59  0000 L BNN
-F 2 "main_new:E5-8,5" H 7300 3700 50  0001 C CNN
-F 3 "" H 7300 3700 50  0001 C CNN
-	1    7300 3700
-	0    1    1    0
-$EndComp
-$Comp
 L main_new-eagle-import:C-EU050-030X075 C3
 U 1 1 30898867
@@
 F 0 "C3" H 6360 4015 59  0000 L BNN
 F 1 "15n" H 6360 3815 59  0000 L BNN
-F 2 "main_new:C050-030X075" H 6300 4000 50  0001 C CNN
+F 2 "Capacitor_SMD:C_0805_2012Metric_Pad1.15x1.40mm_HandSolder" H 6300 4000 50  0001 C CNN
 F 3 "" H 6300 4000 50  0001 C CNN
 	1    6300 4000
@@
 U 1 1 BB1807DC
 P 7200 4000
-F 0 "C4" H 7260 4015 59  0000 L BNN
-F 1 "15n" H 7260 3815 59  0000 L BNN
-F 2 "main_new:C050-030X075" H 7200 4000 50  0001 C CNN
+F 0 "C4" H 7050 4050 59  0000 L BNN
+F 1 "15n" H 7050 3800 59  0000 L BNN
+F 2 "Capacitor_SMD:C_0805_2012Metric_Pad1.15x1.40mm_HandSolder" H 7200 4000 50  0001 C CNN
 F 3 "" H 7200 4000 50  0001 C CNN
 	1    7200 4000
@@
 F 0 "C5" H 6360 4615 59  0000 L BNN
 F 1 "15n" H 6360 4415 59  0000 L BNN
-F 2 "main_new:C050-030X075" H 6300 4600 50  0001 C CNN
+F 2 "Capacitor_SMD:C_0805_2012Metric_Pad1.15x1.40mm_HandSolder" H 6300 4600 50  0001 C CNN
 F 3 "" H 6300 4600 50  0001 C CNN
 	1    6300 4600
@@
 F 0 "C6" H 7360 4615 59  0000 L BNN
 F 1 "15n" H 7360 4415 59  0000 L BNN
-F 2 "main_new:C050-030X075" H 7300 4600 50  0001 C CNN
+F 2 "Capacitor_SMD:C_0805_2012Metric_Pad1.15x1.40mm_HandSolder" H 7300 4600 50  0001 C CNN
 F 3 "" H 7300 4600 50  0001 C CNN
 	1    7300 4600
 	0    1    1    0
-$EndComp
-$Comp
-L main_new-eagle-import:R-EU_0411_12 R1
-U 1 1 23FCBBB2
-P 6500 4300
-F 0 "R1" H 6350 4359 59  0000 L BNN
-F 1 "8/0.8/5.0" H 6350 4170 59  0000 L BNN
-F 2 "main_new:0411_12" H 6500 4300 50  0001 C CNN
-F 3 "" H 6500 4300 50  0001 C CNN
-	1    6500 4300
-	0    -1   -1   0
-$EndComp
-$Comp
-L main_new-eagle-import:R-EU_0411_12 R2
-U 1 1 F2C45C0F
-P 7500 4300
-F 0 "R2" H 7350 4359 59  0000 L BNN
-F 1 "8/0.8/5.0" H 7350 4170 59  0000 L BNN
-F 2 "main_new:0411_12" H 7500 4300 50  0001 C CNN
-F 3 "" H 7500 4300 50  0001 C CNN
-	1    7500 4300
-	0    -1   -1   0
 $EndComp
 $Comp
@@
 F 0 "X3" H 6950 5535 59  0000 R TNN
 F 1 "AK500_2" H 6850 5355 59  0000 L BNN
-F 2 "main_new:AK500_2" H 7000 5500 50  0001 C CNN
+F 2 "TerminalBlock_Phoenix:TerminalBlock_Phoenix_PT-1,5-2-5.0-H_1x02_P5.00mm_Horizontal" H 7000 5500 50  0001 C CNN
 F 3 "" H 7000 5500 50  0001 C CNN
 	1    7000 5500
@@
 F 0 "X3" H 7450 5535 59  0000 R TNN
 F 1 "AK500_2" H 7350 5355 59  0000 L BNN
-F 2 "main_new:AK500_2" H 7500 5500 50  0001 C CNN
+F 2 "TerminalBlock_Phoenix:TerminalBlock_Phoenix_PT-1,5-2-5.0-H_1x02_P5.00mm_Horizontal" H 7500 5500 50  0001 C CNN
 F 3 "" H 7500 5500 50  0001 C CNN
 	2    7500 5500
@@
 F 0 "X4" H 5950 5535 59  0000 R TNN
 F 1 "AK500_2" H 5850 5355 59  0000 L BNN
-F 2 "main_new:AK500_2" H 6000 5500 50  0001 C CNN
+F 2 "TerminalBlock_Phoenix:TerminalBlock_Phoenix_PT-1,5-2-5.0-H_1x02_P5.00mm_Horizontal" H 6000 5500 50  0001 C CNN
 F 3 "" H 6000 5500 50  0001 C CNN
 	1    6000 5500
@@
 F 0 "X4" H 6450 5535 59  0000 R TNN
 F 1 "AK500_2" H 6350 5355 59  0000 L BNN
-F 2 "main_new:AK500_2" H 6500 5500 50  0001 C CNN
+F 2 "TerminalBlock_Phoenix:TerminalBlock_Phoenix_PT-1,5-2-5.0-H_1x02_P5.00mm_Horizontal" H 6500 5500 50  0001 C CNN
 F 3 "" H 6500 5500 50  0001 C CNN
 	2    6500 5500
@@
 	-1   0    0    -1
 $EndComp
+$Comp
+L Device:L_Small L1
+U 1 1 5F60B631
+P 6500 4300
+F 0 "L1" H 6548 4346 50  0000 L CNN
+F 1 "130nH" H 6548 4255 50  0000 L CNN
+F 2 "Lib:XEL3520131MEB" H 6500 4300 50  0001 C CNN
+F 3 "~" H 6500 4300 50  0001 C CNN
+	1    6500 4300
+	1    0    0    -1
+$EndComp
+$Comp
+L Device:L_Small L2
+U 1 1 5F60CB9F
+P 7500 4300
+F 0 "L2" H 7548 4346 50  0000 L CNN
+F 1 "130nH" H 7548 4255 50  0000 L CNN
+F 2 "Lib:XEL3520131MEB" H 7500 4300 50  0001 C CNN
+F 3 "~" H 7500 4300 50  0001 C CNN
+	1    7500 4300
+	1    0    0    -1
+$EndComp
+Wire Wire Line
+	7500 4000 7500 4200
+Wire Wire Line
+	7500 4400 7500 4600
+Wire Wire Line
+	6500 4400 6500 4600
+Wire Wire Line
+	6500 4000 6500 4200
+$Comp
+L power:+15V #PWR0101
+U 1 1 5F61CC74
+P 1300 3250
+F 0 "#PWR0101" H 1300 3100 50  0001 C CNN
+F 1 "+15V" H 1315 3423 50  0000 C CNN
+F 2 "" H 1300 3250 50  0001 C CNN
+F 3 "" H 1300 3250 50  0001 C CNN
+	1    1300 3250
+	-1   0    0    1
+$EndComp
+$Comp
+L power:+15V #PWR0102
+U 1 1 5F61CDBB
+P 3850 3950
+F 0 "#PWR0102" H 3850 3800 50  0001 C CNN
+F 1 "+15V" H 3865 4123 50  0000 C CNN
+F 2 "" H 3850 3950 50  0001 C CNN
+F 3 "" H 3850 3950 50  0001 C CNN
+	1    3850 3950
+	1    0    0    -1
+$EndComp
+$Comp
+L power:PWR_FLAG #FLG0101
+U 1 1 5F61F9D8
+P 1750 3200
+F 0 "#FLG0101" H 1750 3275 50  0001 C CNN
+F 1 "PWR_FLAG" H 1750 3373 50  0000 C CNN
+F 2 "" H 1750 3200 50  0001 C CNN
+F 3 "~" H 1750 3200 50  0001 C CNN
+	1    1750 3200
+	1    0    0    -1
+$EndComp
+Connection ~ 1750 3200
+$Comp
+L power:PWR_FLAG #FLG0102
+U 1 1 5F62081C
+P 1300 3200
+F 0 "#FLG0102" H 1300 3275 50  0001 C CNN
+F 1 "PWR_FLAG" H 1300 3373 50  0000 C CNN
+F 2 "" H 1300 3200 50  0001 C CNN
+F 3 "~" H 1300 3200 50  0001 C CNN
+	1    1300 3200
+	1    0    0    -1
+$EndComp
+Wire Wire Line
+	1300 3200 1300 3250
+$Comp
+L power:PWR_FLAG #FLG0103
+U 1 1 5F620827
+P 1300 3200
+F 0 "#FLG0103" H 1300 3275 50  0001 C CNN
+F 1 "PWR_FLAG" H 1300 3373 50  0000 C CNN
+F 2 "" H 1300 3200 50  0001 C CNN
+F 3 "~" H 1300 3200 50  0001 C CNN
+	1    1300 3200
+	1    0    0    -1
+$EndComp
+Connection ~ 1300 3200
+$Comp
+L power:+15V #PWR0103
+U 1 1 5F6224FF
+P 5000 4700
+F 0 "#PWR0103" H 5000 4550 50  0001 C CNN
+F 1 "+15V" H 5015 4873 50  0000 C CNN
+F 2 "" H 5000 4700 50  0001 C CNN
+F 3 "" H 5000 4700 50  0001 C CNN
+	1    5000 4700
+	1    0    0    -1
+$EndComp
+Wire Wire Line
+	6500 2800 6500 3700
+Connection ~ 6500 3700
+Wire Wire Line
+	6500 3700 6500 4000
+$Comp
+L Device:CP_Small C1
+U 1 1 5F628895
+P 6200 3700
+F 0 "C1" V 5975 3700 50  0000 C CNN
+F 1 "10uF" V 6066 3700 50  0000 C CNN
+F 2 "Capacitor_Tantalum_SMD:CP_EIA-7132-28_AVX-C_Pad2.72x3.50mm_HandSolder" H 6200 3700 50  0001 C CNN
+F 3 "~" H 6200 3700 50  0001 C CNN
+	1    6200 3700
+	0    1    1    0
+$EndComp
+$Comp
+L Device:CP_Small C2
+U 1 1 5F628F69
+P 7200 3700
+F 0 "C2" V 6975 3700 50  0000 C CNN
+F 1 "10uF" V 7066 3700 50  0000 C CNN
+F 2 "Capacitor_Tantalum_SMD:CP_EIA-7132-28_AVX-C_Pad2.72x3.50mm_HandSolder" H 7200 3700 50  0001 C CNN
+F 3 "~" H 7200 3700 50  0001 C CNN
+	1    7200 3700
+	0    1    1    0
+$EndComp
+Wire Wire Line
+	7300 3700 7500 3700
+Wire Wire Line
+	6300 3700 6500 3700
 $EndSCHEMATC
